File: ECAD/Metro Tracker PCB.kicad_sch (KiCad schematic)
At the start: 7 parts, among them IC1 FT230XS-R, IC2 LM1117MPX-3.3_NOPB

Commit message: schematic stuff
Parts:
- removed IC1: FT230XS-R, SOP64P599X175-16N, symbol FT230XS-R:FT230XS-R
- removed J?: USB4125-GF-A-0190, USB4125GFA0190, symbol USB4125-GF-A-0190:USB4125-GF-A-0190
- removed R? (x2): 5.1k, symbol Device:R
- added C3: 22uF/25V(20%), symbol Device:C
- added C4: 0.1uF/50V(10%), symbol Device:C
- added D1: RED LED, symbol Device:LED
- added D2: 1N5819HW-7-F, SOD3716X145N, symbol 1N5819HW-7-F:1N5819HW-7-F
- added D3, D4: ESD5Z5V0, SODFL1608X70N, symbol ESD5Z5V0:ESD5Z5V0
- added IC1: ESP32-S3-WROOM-1-N16R2, ESP32S3WROOM1N16R2, symbol ESP32-S3-WROOM-1-N16R2:ESP32-S3-WROOM-1-N16R2
- added J1: USB4110-GF-A, USB4110GFA, symbol USB4110-GF-A:USB4110-GF-A
- added R1: 2k, symbol Device:R
- added R2, R3: 5.1k, symbol Device:R
- C1: value C -> 10 uF/10V
- C2: value 10 uF -> 10 uF/10V
Connections:
- net +5V: now also C2.1, IC2.3 (INPUT), D2.2 (A), R1.1
- net GND: now also C3.2, C4.2, D1.1 (K), D3.2 (A), D4.2 (A), IC1.1 (GND_1), IC1.13 (IO19), IC1.14 (IO20), J1.A1 (GND), J1.A12 (GND), J1.B1 (GND), J1.B12 (GND), J1.MP1, J1.MP2, J1.MP3, J1.MP4, R2.1, R3.2
- net +3.3V: now reaches C1.1, IC2.2 (OUTPUT), IC2.4 (VOUT)
- net +3.3V: now also C3.1, C4.1, IC1.2 (3V3)
- new net: J1.A5 (CC1), R2.2
- new net: J1.B5 (CC2), R3.1
- new net: D1.2 (A), R1.2
- new net D+: D3.1 (K), J1.A6 (Dp1), J1.B6 (Dp2)
- new net D-: D4.1 (K), J1.A7 (Dn1), J1.B7 (Dn2)
- new net VBUS: D2.1 (K), J1.A4 (VBUS), J1.A9 (VBUS), J1.B4 (VBUS), J1.B9 (VBUS)
- no-connect marks 0 -> 2
Other:
- note added: "ESD Protection"
- note added: "ESP32-S3:"
- note added: "Power Supply ESP32"
- note added: "Reverse Voltage Protection"
- note removed: "ESP32:"
- note removed: "Power Supply: ESP32 + Perfs"
- note removed: "USB2UART Bridge:"
- moved on the sheet: C2, IC2
